File: pcb/mcu.kicad_sch (KiCad schematic)
At the start: 32 parts, among them J1 Conn_01x02_Pin, SW1 SW_Push, SW2 SW_SPDT, U1 STM32H750VBTx, U2 W25Q64JVSSIQ_C179171, U3 TLV1117LV33DCYR, Y1 25 MHz

Commit message: [bom] pcb components and [pcb] assign footprints
Parts:
- added SW3: SW_SPDT, Button_Switch_THT:SW_Slide-03_Wuerth-WS-SLTV_10x2.5x6.4_P2.54mm, symbol Switch:SW_SPDT
- C1: renamed from C2; footprint (none) -> Capacitor_SMD:C_0805_2012Metric_Pad1.18x1.45mm_HandSolder
- C10: renamed from C21; footprint (none) -> Capacitor_SMD:C_0603_1608Metric_Pad1.08x0.95mm_HandSolder
- C11: renamed from C4; footprint (none) -> Capacitor_SMD:C_0805_2012Metric_Pad1.18x1.45mm_HandSolder
- C12: renamed from C5; footprint (none) -> Capacitor_SMD:C_0805_2012Metric_Pad1.18x1.45mm_HandSolder
- C13: renamed from C6; footprint (none) -> Capacitor_SMD:C_0805_2012Metric_Pad1.18x1.45mm_HandSolder
- C14: renamed from C7; footprint (none) -> Capacitor_SMD:C_0805_2012Metric_Pad1.18x1.45mm_HandSolder
- C15: renamed from C8; footprint (none) -> Capacitor_SMD:C_0805_2012Metric_Pad1.18x1.45mm_HandSolder
- C16: renamed from C13; footprint (none) -> Capacitor_SMD:C_0805_2012Metric_Pad1.18x1.45mm_HandSolder
- C17: renamed from C14; footprint (none) -> Capacitor_SMD:C_0805_2012Metric_Pad1.18x1.45mm_HandSolder
- C2: renamed from C3; footprint (none) -> Capacitor_SMD:C_0805_2012Metric_Pad1.18x1.45mm_HandSolder
- C3: renamed from C9; footprint (none) -> Capacitor_SMD:C_0805_2012Metric_Pad1.18x1.45mm_HandSolder
- C4: renamed from C10; footprint (none) -> Capacitor_SMD:C_0805_2012Metric_Pad1.18x1.45mm_HandSolder
- C5: renamed from C11; value 1 uF -> 1uF; footprint (none) -> Capacitor_SMD:C_0805_2012Metric_Pad1.18x1.45mm_HandSolder
- C6: renamed from C1; footprint (none) -> Capacitor_SMD:C_0805_2012Metric_Pad1.18x1.45mm_HandSolder
- C7: renamed from C12; footprint (none) -> Capacitor_SMD:C_0805_2012Metric_Pad1.18x1.45mm_HandSolder
- C8: renamed from C15; footprint (none) -> Capacitor_SMD:C_0805_2012Metric_Pad1.18x1.45mm_HandSolder
- C9: renamed from C20; footprint (none) -> Capacitor_SMD:C_0603_1608Metric_Pad1.08x0.95mm_HandSolder
- FB1: value FCM1608KF-601T05 -> 601T05; footprint (none) -> Inductor_SMD:L_0603_1608Metric_Pad1.05x0.95mm_HandSolder
- J1: footprint (none) -> Connector_JST:JST_XH_B2B-XH-A_1x02_P2.50mm_Vertical
- R1: footprint (none) -> Resistor_SMD:R_0805_2012Metric_Pad1.20x1.40mm_HandSolder
- R2: renamed from R11; footprint (none) -> Resistor_SMD:R_0805_2012Metric_Pad1.20x1.40mm_HandSolder
- R3: renamed from R10; value 10K -> 10k; footprint (none) -> Resistor_SMD:R_0805_2012Metric_Pad1.20x1.40mm_HandSolder
- SW1: renamed from SW2; footprint (none) -> Button_Switch_THT:SW_Slide-03_Wuerth-WS-SLTV_10x2.5x6.4_P2.54mm
- SW2: renamed from SW1; footprint (none) -> Button_Switch_THT:SW_PUSH_6mm
- TP1: renamed from TP4; footprint (none) -> TestPoint:TestPoint_Pad_D2.0mm; now left out of the parts list
- TP2: renamed from TP3; footprint (none) -> TestPoint:TestPoint_Pad_D2.0mm; now left out of the parts list
- TP3: renamed from TP2; footprint (none) -> TestPoint:TestPoint_Pad_D2.0mm; now left out of the parts list
- TP4: renamed from TP1; footprint (none) -> TestPoint:TestPoint_Pad_D2.0mm; now left out of the parts list
- U2: footprint lcsc:SOIC-8_L5.3-W5.3-P1.27-LS8.0-BL -> Package_SO:SOIC-8_5.3x5.3mm_P1.27mm
- Y1: footprint (none) -> Crystal:Crystal_SMD_3225-4Pin_3.2x2.5mm_HandSoldering
- renumbered U3 to U1, U1 to U3
Connections:
- net +3.3V: now also SW3.3 (C)
- net GND: now also SW3.1 (A); no longer R3.1
- new net: R3.1, SW3.2 (B)
Other:
- note added: "Microcontroller Unit"
- note removed: "MCU"
- moved on the sheet: C10, C8, C9, R3, SW2, TP3, TP4, Y1
