File: pcb/peripherals.kicad_sch (KiCad schematic)
At the start: 26 parts, among them J2 Conn_02x11_Odd_Even, SW1 SW_Push, SW3 SW_Push, U4 BMP388, U5 NRF24L01_Breakout, U7 BMI270, U8 HYCW110-TF10-180B

Commit message: [pcb] switch bmi270 to SPI, wire interrupt pins and SD chip detect
Parts:
- removed R16, R17: 2.2k, Resistor_SMD:R_0805_2012Metric_Pad1.20x1.40mm_HandSolder, symbol Device:R
- removed R18, R19: 100k, Resistor_SMD:R_0805_2012Metric_Pad1.20x1.40mm_HandSolder, symbol Device:R
- added J3: Conn_01x04_MountingPin, Connector_JST:JST_SH_BM04B-SRSS-TB_1x04-1MP_P1.00mm_Vertical, symbol Connector_Generic_MountingPin:Conn_01x04_MountingPin
Connections:
- net +BATT: now also J3.1 (Pin_1)
- net GND: now also J3.2 (Pin_2), J3.MP (MountPin); no longer U8.9 (CD)
- net SPI4_MISO: now reaches U7.1 (SDO)
- net IMU_CS: now reaches U7.12 (CSB)
- net IMU_INT1: now reaches U7.4 (INT1)
- net NRF_IRQ: now reaches U5.8 (IRQ)
- net CS_SD renamed SD_CS
- net IMU_SCL renamed SPI4_SCK
- net IMU_SDA renamed SPI4_MOSI
- new net SD_CD: U8.9 (CD)
- new net UART4_RX: J3.3 (Pin_3)
- new net UART4_TX: J3.4 (Pin_4)
- no-connect marks 9 -> 7
