File: controller/pcb/controller.kicad_pcb (KiCad board)
At the start: 2 copper layers, 89.1 x 49.9 mm, 31 parts, among them J1 Conn_01x10_Pin, SW1 SW_Push, SW2 SW_Push, SW3 SW_Push, SW4 SW_Push, U1 PS5, U2 PS5, U3 NRF24L01_Breakout, U4 ESP32C3-SUPERMINI, U5 74HC148

Commit message: [bom] tax + shipping and [controller] add silkscreen
Parts:
- added G***: LOGO, LOGO, B.Cu at (137.7, 70.9)
Other:
- board text added: "0123abc"
- board text added: "@TheScientist101"
- board text added: "@grimsteel"
- board text added: "JLCJLCJLCJLC"
- board text added: "astra"
- board text added: "github.com/TheScientist101/astra"

Commit message: [pcb] update commit silkscreen
Other:
- board text added: "09fc4c9"
- board text removed: "0123abc"
