File: drone/pcb-v2/motor-controller.kicad_sch (KiCad schematic)
At the start: 24 parts, among them M1 Motor_DC, M2 Motor_DC, M3 Motor_DC, M4 Motor_DC, Q1 AO3400A, Q2 AO3400A, Q3 AO3400A, Q4 AO3400A

Commit message: [pcb] schematic v2: footprint/part assignments
Parts:
- C1: renamed from C18; now fitted; now left out of the parts list
- C2: renamed from C19; now fitted; now left out of the parts list
- C3: renamed from C20; now fitted; now left out of the parts list
- C4: renamed from C21; now fitted; now left out of the parts list
- D1, D2, D3, D4: footprint Diode_SMD:D_SOD-323_HandSoldering -> Diode_SMD:D_SOD-323; LCSC (none) -> C2128
- M1, M2, M3, M4: now left out of the parts list
- Q1, Q2, Q3, Q4: footprint Package_TO_SOT_SMD:SOT-23_Handsoldering -> Package_TO_SOT_SMD:SOT-23-3; LCSC (none) -> C20917
- R1: renamed from R4; footprint Resistor_SMD:R_0805_2012Metric_Pad1.20x1.40mm_HandSolder -> Resistor_SMD:R_0805_2012Metric; LCSC (none) -> C17557
- R2: renamed from R5; footprint Resistor_SMD:R_0805_2012Metric_Pad1.20x1.40mm_HandSolder -> Resistor_SMD:R_0805_2012Metric; LCSC (none) -> C17557
- R3: renamed from R6; footprint Resistor_SMD:R_0805_2012Metric_Pad1.20x1.40mm_HandSolder -> Resistor_SMD:R_0805_2012Metric; LCSC (none) -> C17414
- R4: renamed from R7; footprint Resistor_SMD:R_0805_2012Metric_Pad1.20x1.40mm_HandSolder -> Resistor_SMD:R_0805_2012Metric; LCSC (none) -> C17414
- R5: renamed from R8; footprint Resistor_SMD:R_0805_2012Metric_Pad1.20x1.40mm_HandSolder -> Resistor_SMD:R_0805_2012Metric; LCSC (none) -> C17557
- R6: renamed from R9; footprint Resistor_SMD:R_0805_2012Metric_Pad1.20x1.40mm_HandSolder -> Resistor_SMD:R_0805_2012Metric; LCSC (none) -> C17557
- R7: renamed from R10; footprint Resistor_SMD:R_0805_2012Metric_Pad1.20x1.40mm_HandSolder -> Resistor_SMD:R_0805_2012Metric; LCSC (none) -> C17414
- R8: renamed from R11; footprint Resistor_SMD:R_0805_2012Metric_Pad1.20x1.40mm_HandSolder -> Resistor_SMD:R_0805_2012Metric; LCSC (none) -> C17414
